Commit message: Added ground truth to the DJI F450 quadcopter model

File: models/quad_f450_camera/urdf/component_snippets.xacro (robot description, xacro)
@@ -141,4 +141,17 @@
         <biasCorrelationTime>${bias_correlation_time}</biasCorrelationTime>
         <magTopic>${mag_topic}</magTopic>
+      </plugin>
+    </gazebo>
+  </xacro:macro>
+  <!-- Macro to add Ground Truth plugin -->
+  <xacro:macro name="ground_truth_plugin_macro" params="base pub_rate groundt_topic">
+    <gazebo>
+      <plugin name="ground_truth" filename="libgazebo_ros_p3d.so">
+        <frameName>map</frameName>
+		<bodyName>${base}</bodyName>
+		<topicName>${groundt_topic}</topicName>
+		<updateRate>${pub_rate}</updateRate>
+		<xyzOffset>0 0 -0.1975016</xyzOffset>
+		<rpyOffset>0 0 0</rpyOffset>
       </plugin>
     </gazebo>

File: models/quad_f450_camera/urdf/quad_base.xacro (robot description, xacro)
@@ -68,4 +68,11 @@
     >
   </xacro:barometer_plugin_macro>
+  <!-- Instantiate GroundTruth plugin. -->
+  <xacro:ground_truth_plugin_macro
+    base="base_link"
+    pub_rate="30"
+    groundt_topic="/odom"
+    >
+  </xacro:ground_truth_plugin_macro>
   <xacro:if value="$(arg enable_mavlink_interface)">
   <!-- Instantiate mavlink telemetry interface. -->
